Commit message: fix the amcl launch file and add more parameters

File: chaser_robot/urdf/chaser_robot.xacro (robot description, xacro)
@@ -34,5 +34,5 @@
       <material name="black"/>
     </visual>
-    <!--collision name='front_caster_collision'>
+    <collision name='front_caster_collision'>
       <origin xyz="0.15 0 -0.05" rpy=" 0 0 0"/>
       <geometry>
@@ -42,4 +42,16 @@
     <visual name='front_caster_visual'>
       <origin xyz="0.15 0 -0.05" rpy=" 0 0 0"/>
+      <geometry>
+        <sphere radius="0.05"/>
+      </geometry>
+    </visual>
+     <collision name='back_caster_collision'>
+      <origin xyz="-0.15 0 -0.05" rpy=" 0 0 0"/>
+      <geometry>
+        <sphere radius="0.0499"/>
+      </geometry>
+    </collision>
+    <visual name='back_caster_visual'>
+      <origin xyz="-0.15 0 -0.05" rpy=" 0 0 0"/>
       <geometry>
         <sphere radius="0.05"/>
@@ -50,17 +62,17 @@
       <mass value="5.0"/>
       <inertia ixx="0.1" ixy="0.0" ixz="0.0" iyy="0.1" iyz="0.0" izz="0.1"/>
-    </inertial-->
-  </link>
-<link name="F_left_wheel">
-    <collision name='F_left_wheel_collision'>
-      <origin xyz="0 0 0" rpy=" 0 1.5705 1.5705"/>
-      <geometry>
-        <cylinder radius="0.08" length="0.05"/>
-      </geometry>
-    </collision>
-    <visual name='F_left_wheel_visual'>
-      <origin xyz="0 0 0" rpy=" 0 1.5705 1.5705"/>
-      <geometry>
-        <cylinder radius="0.08" length="0.05"/>
+    </inertial>
+  </link>
+  <link name="left_wheel">
+    <collision name='left_wheel_collision'>
+      <origin xyz="0 0 0" rpy=" 0 1.5705 1.5705"/>
+      <geometry>
+        <cylinder radius="0.1" length="0.05"/>
+      </geometry>
+    </collision>
+    <visual name='left_wheel_visual'>
+      <origin xyz="0 0 0" rpy=" 0 1.5705 1.5705"/>
+      <geometry>
+        <cylinder radius="0.1" length="0.05"/>
       </geometry>
       <material name="blue"/>
@@ -72,15 +84,15 @@
     </inertial>
   </link>
-  <link name="F_right_wheel">
-    <collision name='F_right_wheel_collision'>
-      <origin xyz="0 0 0" rpy=" 0 1.5705 1.5705"/>
-      <geometry>
-        <cylinder radius="0.08" length="0.05"/>
-      </geometry>
-    </collision>
-    <visual name='F_right_wheel_visual'>
-      <origin xyz="0 0 0" rpy=" 0 1.5705 1.5705"/>
-      <geometry>
-        <cylinder radius="0.08" length="0.05"/>
+  <link name="right_wheel">
+    <collision name='right_wheel_collision'>
+      <origin xyz="0 0 0" rpy=" 0 1.5705 1.5705"/>
+      <geometry>
+        <cylinder radius="0.1" length="0.05"/>
+      </geometry>
+    </collision>
+    <visual name='right_wheel_visual'>
+      <origin xyz="0 0 0" rpy=" 0 1.5705 1.5705"/>
+      <geometry>
+        <cylinder radius="0.1" length="0.05"/>
       </geometry>
       <material name="blue"/>
@@ -92,47 +104,7 @@
     </inertial>
   </link>
-  <link name="B_left_wheel">
-    <collision name='B_left_wheel_collision'>
-      <origin xyz="0 0 0" rpy=" 0 1.5705 1.5705"/>
-      <geometry>
-        <cylinder radius="0.08" length="0.05"/>
-      </geometry>
-    </collision>
-    <visual name='B_left_wheel_visual'>
-      <origin xyz="0 0 0" rpy=" 0 1.5705 1.5705"/>
-      <geometry>
-        <cylinder radius="0.08" length="0.05"/>
-      </geometry>
-      <material name="blue"/>
-    </visual>
-    <inertial>
-      <origin xyz="0.0 0.0 0.0" rpy="0.0 1.5707 1.5707"/>
-      <mass value="5.0"/>
-      <inertia ixx="0.1" ixy="0.0" ixz="0.0" iyy="0.1" iyz="0.0" izz="0.1"/>
-    </inertial>
-  </link>
-  <link name="B_right_wheel">
-    <collision name='B_right_wheel_collision'>
-      <origin xyz="0 0 0" rpy=" 0 1.5705 1.5705"/>
-      <geometry>
-        <cylinder radius="0.08" length="0.05"/>
-      </geometry>
-    </collision>
-    <visual name='B_right_wheel_visual'>
-      <origin xyz="0 0 0" rpy=" 0 1.5705 1.5705"/>
-      <geometry>
-        <cylinder radius="0.08" length="0.05"/>
-      </geometry>
-      <material name="blue"/>
-    </visual>
-    <inertial>
-      <origin xyz="0.0 0.0 0.0" rpy="0.0 1.5707 1.5707"/>
-      <mass value="5.0"/>
-      <inertia ixx="0.1" ixy="0.0" ixz="0.0" iyy="0.1" iyz="0.0" izz="0.1"/>
-    </inertial>
-  </link>
-<joint type="continuous" name="F_left_wheel_hinge">
-    <origin xyz="0.13 0.15 0" rpy="0 0 0"/>
-    <child link="F_left_wheel"/>
+  <joint type="continuous" name="left_wheel_hinge">
+    <origin xyz="0 0.15 0" rpy="0 0 0"/>
+    <child link="left_wheel"/>
     <parent link="chassis"/>
     <axis xyz="0 1 0" rpy="0 0 0"/>
@@ -140,23 +112,7 @@
     <dynamics damping="1.0" friction="1.0"/>
   </joint>
-  <joint type="continuous" name="F_right_wheel_hinge">
-    <origin xyz="0.13 -0.15 0" rpy="0 0 0"/>
-    <child link="F_right_wheel"/>
-    <parent link="chassis"/>
-    <axis xyz="0 1 0" rpy="0 0 0"/>
-    <limit effort="10000" velocity="1000"/>
-    <dynamics damping="1.0" friction="1.0"/>
-  </joint>
-  <joint type="continuous" name="B_left_wheel_hinge">
-    <origin xyz="-0.15 0.15 0" rpy="0 0 0"/>
-    <child link="B_left_wheel"/>
-    <parent link="chassis"/>
-    <axis xyz="0 1 0" rpy="0 0 0"/>
-    <limit effort="10000" velocity="1000"/>
-    <dynamics damping="1.0" friction="1.0"/>
-  </joint>
-  <joint type="continuous" name="B_right_wheel_hinge">
-    <origin xyz="-0.15 -0.15 0" rpy="0 0 0"/>
-    <child link="B_right_wheel"/>
+  <joint type="continuous" name="right_wheel_hinge">
+    <origin xyz="0 -0.15 0" rpy="0 0 0"/>
+    <child link="right_wheel"/>
     <parent link="chassis"/>
     <axis xyz="0 1 0" rpy="0 0 0"/>
